Commit message: changed to 4 lanes of cars. Need to save imgs now

File: urdfs/agent.urdf (robot description, URDF)
Before this commit: robot random_box, 1 links, 0 joints
Links:
- link box: geometry collision box size=0.9 0.7 0.6; visual box size=0.9 0.7 0.6

File: urdfs/obstacles/obstacle_1.urdf (robot description, URDF)
Before this commit: robot random_box, 1 links, 0 joints
Links:
- link box: geometry collision box size=0.9 0.7 0.6; visual box size=0.9 0.7 0.6

File: urdfs/obstacles/obstacle_10.urdf (robot description, URDF)
Before this commit: robot random_box, 1 links, 0 joints
Links:
- link box: geometry collision box size=0.9 0.7 0.6; visual box size=0.9 0.7 0.6

File: urdfs/obstacles/obstacle_2.urdf (robot description, URDF)
Before this commit: robot random_box, 1 links, 0 joints
Links:
- link box: geometry collision box size=0.9 0.7 0.6; visual box size=0.9 0.7 0.6

File: urdfs/obstacles/obstacle_3.urdf (robot description, URDF)
Before this commit: robot random_box, 1 links, 0 joints
Links:
- link box: geometry collision box size=0.9 0.7 0.6; visual box size=0.9 0.7 0.6

File: urdfs/obstacles/obstacle_4.urdf (robot description, URDF)
Before this commit: robot random_box, 1 links, 0 joints
Links:
- link box: geometry collision box size=0.9 0.7 0.6; visual box size=0.9 0.7 0.6

File: urdfs/obstacles/obstacle_5.urdf (robot description, URDF)
Before this commit: robot random_box, 1 links, 0 joints
Links:
- link box: geometry collision box size=0.9 0.7 0.6; visual box size=0.9 0.7 0.6

File: urdfs/obstacles/obstacle_6.urdf (robot description, URDF)
Before this commit: robot random_box, 1 links, 0 joints
Links:
- link box: geometry collision box size=0.9 0.7 0.6; visual box size=0.9 0.7 0.6

File: urdfs/obstacles/obstacle_7.urdf (robot description, URDF)
Before this commit: robot random_box, 1 links, 0 joints
Links:
- link box: geometry collision box size=0.9 0.7 0.6; visual box size=0.9 0.7 0.6

File: urdfs/obstacles/obstacle_8.urdf (robot description, URDF)
Before this commit: robot random_box, 1 links, 0 joints
Links:
- link box: geometry collision box size=0.9 0.7 0.6; visual box size=0.9 0.7 0.6

File: urdfs/obstacles/obstacle_9.urdf (robot description, URDF)
Before this commit: robot random_box, 1 links, 0 joints
Links:
- link box: geometry collision box size=0.9 0.7 0.6; visual box size=0.9 0.7 0.6

File: urdfs/surroundings/ground.urdf (robot description, URDF)
Before this commit: robot plane_road, 2 links, 1 joints
Links:
- link road: geometry visual box size=4 40 0.001
- link side: geometry visual box size=20 40 0.000001
