Commit message: went back and tried to delete the too big file from upload

File: urdfs/surroundings/background.urdf (robot description, URDF)
Before this commit: robot background_plane, 1 links, 0 joints
Links:
- link background: geometry visual box size=80 20 0.0001

File: urdfs/surroundings/ground.urdf (robot description, URDF)
Before this commit: robot plane_road, 2 links, 1 joints
Links:
- link road: geometry collision box size=4 80 0.001; visual box size=4 80 0.001
- link side: geometry visual box size=40 80 0.000001
