Commit message: fixed simulation environment. Need to work on delta_v in nn

File: urdfs/real_cars/bmw_z4.urdf (robot description, URDF)
Before this commit: robot random_box, 1 links, 0 joints
Links:
- link box: mass 300 -> 5000

File: urdfs/real_cars/fiat_500.urdf (robot description, URDF)
Before this commit: robot random_box, 1 links, 0 joints
Links:
- link box: mass 200 -> 5000

File: urdfs/real_cars/honda.urdf (robot description, URDF)
Before this commit: robot random_box, 1 links, 0 joints
Links:
- link box: mass 300 -> 5000

File: urdfs/real_cars/mercedes_slk.urdf (robot description, URDF)
Before this commit: robot random_box, 1 links, 0 joints
Links:
- link box: mass 300 -> 5000

File: urdfs/real_cars/van_car.urdf (robot description, URDF)
Before this commit: robot random_box, 1 links, 0 joints
Links:
- link box: mass 700 -> 5000

File: urdfs/real_cars/volga.urdf (robot description, URDF)
Before this commit: robot random_box, 1 links, 0 joints
Links:
- link box: mass 300 -> 5000
